Commit message: updated obstacle avoidance added cnn publisher and updated the modedl to be better

File: install/bot_simulation/share/bot_simulation/model/robot_model.xacro (robot description, xacro)
@@ -151,5 +151,5 @@
     <parent link="body_link"/>
     <child link="camera_link"/>
-    <origin xyz="${camera_length/3.5 + body_link_x_dim/2 } 0 0" rpy="0 0 0"/>
+    <origin xyz="${camera_length/3.5 + body_link_x_dim/2 } 0 ${body_link_z_dim - camera_length*1.5}" rpy="0 0 0"/>
   </joint>
   <link name="camera_link">
