Commit message: feat: add Gazebo environment models, world files, and updated robot launch

File: src/bot_simulation/model/robot_model.xacro (robot description, xacro)
@@ -54,6 +54,6 @@
       </geometry>
       <origin rpy="0 0 0" xyz="0 0 0"/>
-      <material name="pink">
-        <color rgba="0.98 0.75 0.80 1.0"/>
+      <material name="blue">
+        <color rgba="0.0 0.3 0.8 1.0"/>
       </material>
     </visual>
@@ -87,6 +87,6 @@
         <cylinder length="${wheel_link_length}" radius="${wheel_link_radius}"/>
       </geometry>
-      <material name="purple">
-        <color rgba="0.85 0.7 1.0 1.0"/>
+      <material name="black">
+        <color rgba="0.1 0.1 0.1 1.0"/>
       </material>
     </visual>
@@ -113,6 +113,6 @@
         <cylinder length="${wheel_link_length}" radius="${wheel_link_radius}"/>
       </geometry>
-      <material name="purple">
-        <color rgba="0.85 0.7 1.0 1.0"/>
+      <material name="black">
+        <color rgba="0.1 0.1 0.1 1.0"/>
       </material>
     </visual>
@@ -151,5 +151,5 @@
     <parent link="body_link"/>
     <child link="camera_link"/>
-    <origin xyz="${camera_length/3.5 + body_link_x_dim/2 } 0 ${body_link_z_dim - camera_length*1.5}" rpy="0 0 0"/>
+    <origin xyz="${camera_length/3.5 + body_link_x_dim/2 } 0 0" rpy="0 0 0"/>
   </joint>
   <link name="camera_link">
@@ -207,6 +207,6 @@
     <visual>
       <material>
-        <ambient>0.98 0.75 0.80 1.0</ambient>
-        <diffuse>0.98 0.75 0.80 1.0</diffuse>
+        <ambient>0.0 0.3 0.8 1.0</ambient>
+        <diffuse>0.0 0.3 0.8 1.0</diffuse>
       </material>
     </visual>
@@ -217,6 +217,6 @@
     <visual>
       <material>
-        <ambient>0.85 0.7 1.0 1.0</ambient>
-        <diffuse>0.85 0.7 1.0 1.0</diffuse>
+        <ambient>0.1 0.1 0.1 1.0</ambient>
+        <diffuse>0.1 0.1 0.1 1.0</diffuse>
       </material>
     </visual>
@@ -227,6 +227,6 @@
     <visual>
       <material>
-        <ambient>0.85 0.7 1.0 1.0</ambient>
-        <diffuse>0.85 0.7 1.0 1.0</diffuse>
+        <ambient>0.1 0.1 0.1 1.0</ambient>
+        <diffuse>0.1 0.1 0.1 1.0</diffuse>
       </material>
     </visual>

Commit message: final cnn file

File: src/bot_simulation/model/robot_model.xacro (robot description, xacro)
@@ -151,5 +151,5 @@
     <parent link="body_link"/>
     <child link="camera_link"/>
-    <origin xyz="${camera_length/3.5 + body_link_x_dim/2 } 0 0" rpy="0 0 0"/>
+    <origin xyz="${camera_length/3.5 + body_link_x_dim/2 } 0 0.75" rpy="0 0 0"/>
   </joint>
   <link name="camera_link">
